File: Hardware/Lumenati_8-Stick.kicad_pcb (KiCad board)
At the start: 2 copper layers, 56.5 x 14.6 mm, 22 parts, among them J1 CONN_041X04_NO_SILK, J2 CONN_041X04_NO_SILK, U1 APA102, U2 APA102, U3 APA102, U4 APA102, U5 APA102, U6 APA102, U7 APA102, U8 APA102

Commit message: Changed all the names to Lumenati.
Other:
- board text added: "Lumenati 8-Stick"
- board text removed: "HiBeams 8-Stick"
Changed lines of the file:
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@@
   )
   (setup
-    (last_trace_width 1.524)
+    (last_trace_width 0.25)
     (user_trace_width 0.2032)
     (user_trace_width 0.254)
@@
     (effects (font (size 1.5 1.5) (thickness 0.3)))
   )
-  (gr_text "HiBeams 8-Stick" (at 186.69 189.484) (layer Cmts.User)
+  (gr_text "Lumenati 8-Stick" (at 186.69 189.484) (layer Cmts.User)
     (effects (font (size 1.5 1.5) (thickness 0.3)) (justify left))
   )
@@
     (effects (font (size 1.016 1.016) (thickness 0.2032)) (justify mirror))
   )
-  (gr_text "HiBeams 8-Stick" (at 148.8186 103.886) (layer B.SilkS)
+  (gr_text "Lumenati 8-Stick" (at 148.8186 103.886) (layer B.SilkS)
     (effects (font (size 1.5 1.5) (thickness 0.299999)) (justify mirror))
   )
-  (segment (start 177.165 99.06) (end 177.1142 99.0092) (width 1.524) (layer B.Cu) (net 1) (status C00000))
-  (segment (start 177.1142 99.0092) (end 174.5488 99.0092) (width 1.524) (layer B.Cu) (net 1) (status 400000))
+  (segment (start 177.165 99.06) (end 177.1142 99.0092) (width 1.524) (layer B.Cu) (net 1))
+  (segment (start 177.1142 99.0092) (end 174.5488 99.0092) (width 1.524) (layer B.Cu) (net 1))
   (segment (start 174.5488 99.0092) (end 174.5488 99.06) (width 1.524) (layer B.Cu) (net 1))
-  (segment (start 120.65 99.06) (end 120.7008 99.0092) (width 1.524) (layer B.Cu) (net 1) (status C00000))
-  (segment (start 120.7008 99.0092) (end 122.8344 99.0092) (width 1.524) (layer B.Cu) (net 1) (status 400000))
+  (segment (start 120.65 99.06) (end 120.7008 99.0092) (width 1.524) (layer B.Cu) (net 1))
+  (segment (start 120.7008 99.0092) (end 122.8344 99.0092) (width 1.524) (layer B.Cu) (net 1))
   (segment (start 122.8344 99.0092) (end 122.8344 99.06) (width 1.524) (layer B.Cu) (net 1))
   (segment (start 120.65 99.06) (end 122.8344 99.06) (width 0.4064) (layer B.Cu) (net 1))

Commit message: Updated version to v10.
Other:
- board text added: "v10"
- board text removed: "v01"
Changed lines of the file:
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@@
     (links 46)
     (no_connects 0)
-    (area 107.264286 87.292311 239.952514 194.4858)
+    (area 107.264286 87.292311 272.8378 194.5366)
     (thickness 1.6)
-    (drawings 45)
+    (drawings 46)
     (tracks 214)
     (zones 0)
@@
     (pad "" np_thru_hole circle (at 0 0) (size 2.921 2.921) (drill 2.921) (layers *.Cu *.Mask))
   )
+  (gr_text v10 (at 270.6878 193.1416) (layer Cmts.User)
+    (effects (font (size 1.5 1.5) (thickness 0.3)))
+  )
   (dimension 14.605 (width 0.3) (layer Dwgs.User)
     (gr_text "0.5750 in" (at 112.95 100.6475 270) (layer Dwgs.User)
@@
   (gr_arc (start 127.8636 97.79) (end 123.3932 97.79) (angle 90) (layer Edge.Cuts) (width 0.15))
   (gr_arc (start 127.8636 97.7646) (end 127.8636 93.3196) (angle 90) (layer Edge.Cuts) (width 0.15))
-  (gr_text v01 (at 162.8902 98.7044) (layer B.Cu)
+  (gr_text v10 (at 162.8902 98.7044) (layer B.Cu)
     (effects (font (size 0.8128 0.8128) (thickness 0.2032)) (justify mirror))
   )
